Commit message: Fix asset paths

File: ros_pendulum/urdf/robot.xacro (robot description, xacro)
@@ -14,5 +14,5 @@
       <origin xyz="0 0 0" rpy="1.5708 0 -0"/>
       <geometry>
-        <mesh filename="package://assets/housing.stl"/>
+        <mesh filename="package://ros_pendulum/urdf/assets/housing.stl"/>
       </geometry>
       <material name="housing_material">
@@ -23,5 +23,5 @@
       <origin xyz="0 0 0" rpy="1.5708 0 -0"/>
       <geometry>
-        <mesh filename="package://assets/housing.stl"/>
+        <mesh filename="package://ros_pendulum/urdf/assets/housing.stl"/>
       </geometry>
     </collision>
@@ -38,5 +38,5 @@
       <origin xyz="-0 0 0.0392" rpy="-0 1.5708 0"/>
       <geometry>
-        <mesh filename="package://assets/motor_handle.stl"/>
+        <mesh filename="package://ros_pendulum/urdf/assets/motor_handle.stl"/>
       </geometry>
       <material name="motor_handle_material">
@@ -47,5 +47,5 @@
       <origin xyz="-0 0 0.0392" rpy="-0 1.5708 0"/>
       <geometry>
-        <mesh filename="package://assets/motor_handle.stl"/>
+        <mesh filename="package://ros_pendulum/urdf/assets/motor_handle.stl"/>
       </geometry>
     </collision>
@@ -54,5 +54,5 @@
       <origin xyz="0.241369 0 -0.0111" rpy="-0 0 0"/>
       <geometry>
-        <mesh filename="package://assets/bearing.stl"/>
+        <mesh filename="package://ros_pendulum/urdf/assets/bearing.stl"/>
       </geometry>
       <material name="bearing_material">
@@ -63,5 +63,5 @@
       <origin xyz="0.241369 0 -0.0111" rpy="-0 0 0"/>
       <geometry>
-        <mesh filename="package://assets/bearing.stl"/>
+        <mesh filename="package://ros_pendulum/urdf/assets/bearing.stl"/>
       </geometry>
     </collision>
@@ -70,5 +70,5 @@
       <origin xyz="0.241369 0 -0.0111" rpy="-0 0 0"/>
       <geometry>
-        <mesh filename="package://assets/encoder_plate.stl"/>
+        <mesh filename="package://ros_pendulum/urdf/assets/encoder_plate.stl"/>
       </geometry>
       <material name="encoder_plate_material">
@@ -79,5 +79,5 @@
       <origin xyz="0.241369 0 -0.0111" rpy="-0 0 0"/>
       <geometry>
-        <mesh filename="package://assets/encoder_plate.stl"/>
+        <mesh filename="package://ros_pendulum/urdf/assets/encoder_plate.stl"/>
       </geometry>
     </collision>
@@ -86,5 +86,5 @@
       <origin xyz="0.241369 0 -0.0111" rpy="-0 0 0"/>
       <geometry>
-        <mesh filename="package://assets/fixed_handle.stl"/>
+        <mesh filename="package://ros_pendulum/urdf/assets/fixed_handle.stl"/>
       </geometry>
       <material name="fixed_handle_material">
@@ -95,5 +95,5 @@
       <origin xyz="0.241369 0 -0.0111" rpy="-0 0 0"/>
       <geometry>
-        <mesh filename="package://assets/fixed_handle.stl"/>
+        <mesh filename="package://ros_pendulum/urdf/assets/fixed_handle.stl"/>
       </geometry>
     </collision>
@@ -102,5 +102,5 @@
       <origin xyz="0 -0 0.039" rpy="3.14159 1.5708 0"/>
       <geometry>
-        <mesh filename="package://assets/shaft.stl"/>
+        <mesh filename="package://ros_pendulum/urdf/assets/shaft.stl"/>
       </geometry>
       <material name="shaft_material">
@@ -111,5 +111,5 @@
       <origin xyz="0 -0 0.039" rpy="3.14159 1.5708 0"/>
       <geometry>
-        <mesh filename="package://assets/shaft.stl"/>
+        <mesh filename="package://ros_pendulum/urdf/assets/shaft.stl"/>
       </geometry>
     </collision>
@@ -118,5 +118,5 @@
       <origin xyz="0.241369 0 -0.0111" rpy="-0 0 0"/>
       <geometry>
-        <mesh filename="package://assets/fixed_cap.stl"/>
+        <mesh filename="package://ros_pendulum/urdf/assets/fixed_cap.stl"/>
       </geometry>
       <material name="fixed_cap_material">
@@ -127,5 +127,5 @@
       <origin xyz="0.241369 0 -0.0111" rpy="-0 0 0"/>
       <geometry>
-        <mesh filename="package://assets/fixed_cap.stl"/>
+        <mesh filename="package://ros_pendulum/urdf/assets/fixed_cap.stl"/>
       </geometry>
     </collision>
@@ -134,5 +134,5 @@
       <origin xyz="0.241369 0 -0.0111" rpy="-0 0 0"/>
       <geometry>
-        <mesh filename="package://assets/encoder_plate_spacer.stl"/>
+        <mesh filename="package://ros_pendulum/urdf/assets/encoder_plate_spacer.stl"/>
       </geometry>
       <material name="encoder_plate_spacer_material">
@@ -143,5 +143,5 @@
       <origin xyz="0.241369 0 -0.0111" rpy="-0 0 0"/>
       <geometry>
-        <mesh filename="package://assets/encoder_plate_spacer.stl"/>
+        <mesh filename="package://ros_pendulum/urdf/assets/encoder_plate_spacer.stl"/>
       </geometry>
     </collision>
@@ -150,5 +150,5 @@
       <origin xyz="0.241369 0 -0.0111" rpy="-0 0 0"/>
       <geometry>
-        <mesh filename="package://assets/as5600_breakout_board.stl"/>
+        <mesh filename="package://ros_pendulum/urdf/assets/as5600_breakout_board.stl"/>
       </geometry>
       <material name="as5600_breakout_board_material">
@@ -159,5 +159,5 @@
       <origin xyz="0.241369 0 -0.0111" rpy="-0 0 0"/>
       <geometry>
-        <mesh filename="package://assets/as5600_breakout_board.stl"/>
+        <mesh filename="package://ros_pendulum/urdf/assets/as5600_breakout_board.stl"/>
       </geometry>
     </collision>
@@ -166,5 +166,5 @@
       <origin xyz="-0 0 0.0392" rpy="-0 1.5708 0"/>
       <geometry>
-        <mesh filename="package://assets/makerbeam_10mm.stl"/>
+        <mesh filename="package://ros_pendulum/urdf/assets/makerbeam_10mm.stl"/>
       </geometry>
       <material name="makerbeam_10mm_material">
@@ -175,5 +175,5 @@
       <origin xyz="-0 0 0.0392" rpy="-0 1.5708 0"/>
       <geometry>
-        <mesh filename="package://assets/makerbeam_10mm.stl"/>
+        <mesh filename="package://ros_pendulum/urdf/assets/makerbeam_10mm.stl"/>
       </geometry>
     </collision>
@@ -190,5 +190,5 @@
       <origin xyz="0 0 0" rpy="-3.14159 -0 -0"/>
       <geometry>
-        <mesh filename="package://assets/mobile_cap.stl"/>
+        <mesh filename="package://ros_pendulum/urdf/assets/mobile_cap.stl"/>
       </geometry>
       <material name="mobile_cap_material">
@@ -199,5 +199,5 @@
       <origin xyz="0 0 0" rpy="-3.14159 -0 -0"/>
       <geometry>
-        <mesh filename="package://assets/mobile_cap.stl"/>
+        <mesh filename="package://ros_pendulum/urdf/assets/mobile_cap.stl"/>
       </geometry>
     </collision>
@@ -206,5 +206,5 @@
       <origin xyz="0 0 0" rpy="-3.14159 -0 -0"/>
       <geometry>
-        <mesh filename="package://assets/mobile_handle.stl"/>
+        <mesh filename="package://ros_pendulum/urdf/assets/mobile_handle.stl"/>
       </geometry>
       <material name="mobile_handle_material">
@@ -215,5 +215,5 @@
       <origin xyz="0 0 0" rpy="-3.14159 -0 -0"/>
       <geometry>
-        <mesh filename="package://assets/mobile_handle.stl"/>
+        <mesh filename="package://ros_pendulum/urdf/assets/mobile_handle.stl"/>
       </geometry>
     </collision>
@@ -222,5 +222,5 @@
       <origin xyz="0 0 0" rpy="-3.14159 -0 -0"/>
       <geometry>
-        <mesh filename="package://assets/bearing_axe.stl"/>
+        <mesh filename="package://ros_pendulum/urdf/assets/bearing_axe.stl"/>
       </geometry>
       <material name="bearing_axe_material">
@@ -231,5 +231,5 @@
       <origin xyz="0 0 0" rpy="-3.14159 -0 -0"/>
       <geometry>
-        <mesh filename="package://assets/bearing_axe.stl"/>
+        <mesh filename="package://ros_pendulum/urdf/assets/bearing_axe.stl"/>
       </geometry>
     </collision>
@@ -238,5 +238,5 @@
       <origin xyz="0.234 -0 -0.0295" rpy="0 -1.5708 0"/>
       <geometry>
-        <mesh filename="package://assets/makerbeam_10mm.stl"/>
+        <mesh filename="package://ros_pendulum/urdf/assets/makerbeam_10mm.stl"/>
       </geometry>
       <material name="makerbeam_10mm_2_material">
@@ -247,5 +247,5 @@
       <origin xyz="0.234 -0 -0.0295" rpy="0 -1.5708 0"/>
       <geometry>
-        <mesh filename="package://assets/makerbeam_10mm.stl"/>
+        <mesh filename="package://ros_pendulum/urdf/assets/makerbeam_10mm.stl"/>
       </geometry>
     </collision>
@@ -254,5 +254,5 @@
       <origin xyz="0 0 0" rpy="-3.14159 -0 -0"/>
       <geometry>
-        <mesh filename="package://assets/mobile_spacer.stl"/>
+        <mesh filename="package://ros_pendulum/urdf/assets/mobile_spacer.stl"/>
       </geometry>
       <material name="mobile_spacer_material">
@@ -263,5 +263,5 @@
       <origin xyz="0 0 0" rpy="-3.14159 -0 -0"/>
       <geometry>
-        <mesh filename="package://assets/mobile_spacer.stl"/>
+        <mesh filename="package://ros_pendulum/urdf/assets/mobile_spacer.stl"/>
       </geometry>
     </collision>
@@ -270,5 +270,5 @@
       <origin xyz="0 0 0" rpy="-3.14159 -0 -0"/>
       <geometry>
-        <mesh filename="package://assets/magnet_stand.stl"/>
+        <mesh filename="package://ros_pendulum/urdf/assets/magnet_stand.stl"/>
       </geometry>
       <material name="magnet_stand_material">
@@ -279,5 +279,5 @@
       <origin xyz="0 0 0" rpy="-3.14159 -0 -0"/>
       <geometry>
-        <mesh filename="package://assets/magnet_stand.stl"/>
+        <mesh filename="package://ros_pendulum/urdf/assets/magnet_stand.stl"/>
       </geometry>
     </collision>

Commit message: Pendulum works in ROS (except gear ratio)

File: ros_pendulum/urdf/robot.xacro (robot description, xacro)
@@ -293,5 +293,6 @@
   <!-- Joint from housing to shaft -->
   <joint name="gim6010" type="revolute">
-    <origin xyz="0.039 -0 -0" rpy="-0 1.5708 0"/>
+    <!-- I had to change the pitch angle (-180 degrees) -->
+    <origin xyz="0.039 -0 -0" rpy="-0 -1.5708 0"/>
     <parent link="housing"/>
     <child link="shaft"/>
