Commit message: Updated CAD, reduced encoder latency, simulated latency, added action history

File: ros_pendulum/urdf/robot.xacro (robot description, xacro)
@@ -14,5 +14,5 @@
       <origin xyz="0 0 0" rpy="1.5708 0 -0"/>
       <geometry>
-        <mesh filename="package://assets/housing.stl"/>
+        <mesh filename="package://ros_pendulum/urdf/assets/housing.stl"/>
       </geometry>
       <material name="housing_material">
@@ -23,5 +23,5 @@
       <origin xyz="0 0 0" rpy="1.5708 0 -0"/>
       <geometry>
-        <mesh filename="package://assets/housing.stl"/>
+        <mesh filename="package://ros_pendulum/urdf/assets/housing.stl"/>
       </geometry>
     </collision>
@@ -38,5 +38,5 @@
       <origin xyz="-0 0 0.039" rpy="0 1.5708 0"/>
       <geometry>
-        <mesh filename="package://assets/shaft.stl"/>
+        <mesh filename="package://ros_pendulum/urdf/assets/shaft.stl"/>
       </geometry>
       <material name="shaft_material">
@@ -47,5 +47,5 @@
       <origin xyz="-0 0 0.039" rpy="0 1.5708 0"/>
       <geometry>
-        <mesh filename="package://assets/shaft.stl"/>
+        <mesh filename="package://ros_pendulum/urdf/assets/shaft.stl"/>
       </geometry>
     </collision>
@@ -62,5 +62,5 @@
       <origin xyz="-0 -0 0.0437" rpy="-1.5708 1.5708 0"/>
       <geometry>
-        <mesh filename="package://assets/motor_handle.stl"/>
+        <mesh filename="package://ros_pendulum/urdf/assets/motor_handle.stl"/>
       </geometry>
       <material name="motor_handle_material">
@@ -71,5 +71,5 @@
       <origin xyz="-0 -0 0.0437" rpy="-1.5708 1.5708 0"/>
       <geometry>
-        <mesh filename="package://assets/motor_handle.stl"/>
+        <mesh filename="package://ros_pendulum/urdf/assets/motor_handle.stl"/>
       </geometry>
     </collision>
@@ -78,5 +78,5 @@
       <origin xyz="0 0.241369 -0.0096" rpy="0 0 1.5708"/>
       <geometry>
-        <mesh filename="package://assets/bearing.stl"/>
+        <mesh filename="package://ros_pendulum/urdf/assets/bearing.stl"/>
       </geometry>
       <material name="bearing_material">
@@ -87,5 +87,5 @@
       <origin xyz="0 0.241369 -0.0096" rpy="0 0 1.5708"/>
       <geometry>
-        <mesh filename="package://assets/bearing.stl"/>
+        <mesh filename="package://ros_pendulum/urdf/assets/bearing.stl"/>
       </geometry>
     </collision>
@@ -94,5 +94,5 @@
       <origin xyz="0 0.241369 -0.0096" rpy="0 0 1.5708"/>
       <geometry>
-        <mesh filename="package://assets/encoder_plate.stl"/>
+        <mesh filename="package://ros_pendulum/urdf/assets/encoder_plate.stl"/>
       </geometry>
       <material name="encoder_plate_material">
@@ -103,5 +103,5 @@
       <origin xyz="0 0.241369 -0.0096" rpy="0 0 1.5708"/>
       <geometry>
-        <mesh filename="package://assets/encoder_plate.stl"/>
+        <mesh filename="package://ros_pendulum/urdf/assets/encoder_plate.stl"/>
       </geometry>
     </collision>
@@ -110,5 +110,5 @@
       <origin xyz="0 0.241369 -0.0096" rpy="0 0 1.5708"/>
       <geometry>
-        <mesh filename="package://assets/fixed_handle.stl"/>
+        <mesh filename="package://ros_pendulum/urdf/assets/fixed_handle.stl"/>
       </geometry>
       <material name="fixed_handle_material">
@@ -119,5 +119,5 @@
       <origin xyz="0 0.241369 -0.0096" rpy="0 0 1.5708"/>
       <geometry>
-        <mesh filename="package://assets/fixed_handle.stl"/>
+        <mesh filename="package://ros_pendulum/urdf/assets/fixed_handle.stl"/>
       </geometry>
     </collision>
@@ -126,5 +126,5 @@
       <origin xyz="0 0.241369 -0.0096" rpy="0 0 1.5708"/>
       <geometry>
-        <mesh filename="package://assets/fixed_cap.stl"/>
+        <mesh filename="package://ros_pendulum/urdf/assets/fixed_cap.stl"/>
       </geometry>
       <material name="fixed_cap_material">
@@ -135,5 +135,5 @@
       <origin xyz="0 0.241369 -0.0096" rpy="0 0 1.5708"/>
       <geometry>
-        <mesh filename="package://assets/fixed_cap.stl"/>
+        <mesh filename="package://ros_pendulum/urdf/assets/fixed_cap.stl"/>
       </geometry>
     </collision>
@@ -142,5 +142,5 @@
       <origin xyz="0 0.241369 -0.0096" rpy="0 0 1.5708"/>
       <geometry>
-        <mesh filename="package://assets/encoder_plate_spacer.stl"/>
+        <mesh filename="package://ros_pendulum/urdf/assets/encoder_plate_spacer.stl"/>
       </geometry>
       <material name="encoder_plate_spacer_material">
@@ -151,5 +151,5 @@
       <origin xyz="0 0.241369 -0.0096" rpy="0 0 1.5708"/>
       <geometry>
-        <mesh filename="package://assets/encoder_plate_spacer.stl"/>
+        <mesh filename="package://ros_pendulum/urdf/assets/encoder_plate_spacer.stl"/>
       </geometry>
     </collision>
@@ -158,5 +158,5 @@
       <origin xyz="0 0.241369 -0.0096" rpy="0 0 1.5708"/>
       <geometry>
-        <mesh filename="package://assets/as5600_breakout_board.stl"/>
+        <mesh filename="package://ros_pendulum/urdf/assets/as5600_breakout_board.stl"/>
       </geometry>
       <material name="as5600_breakout_board_material">
@@ -167,5 +167,5 @@
       <origin xyz="0 0.241369 -0.0096" rpy="0 0 1.5708"/>
       <geometry>
-        <mesh filename="package://assets/as5600_breakout_board.stl"/>
+        <mesh filename="package://ros_pendulum/urdf/assets/as5600_breakout_board.stl"/>
       </geometry>
     </collision>
@@ -174,5 +174,5 @@
       <origin xyz="0 -0 0.0437" rpy="-1.5708 1.5708 0"/>
       <geometry>
-        <mesh filename="package://assets/makerbeam_10mm.stl"/>
+        <mesh filename="package://ros_pendulum/urdf/assets/makerbeam_10mm.stl"/>
       </geometry>
       <material name="makerbeam_10mm_material">
@@ -183,5 +183,5 @@
       <origin xyz="0 -0 0.0437" rpy="-1.5708 1.5708 0"/>
       <geometry>
-        <mesh filename="package://assets/makerbeam_10mm.stl"/>
+        <mesh filename="package://ros_pendulum/urdf/assets/makerbeam_10mm.stl"/>
       </geometry>
     </collision>
@@ -198,5 +198,5 @@
       <origin xyz="0 0 0" rpy="3.14159 0 0"/>
       <geometry>
-        <mesh filename="package://assets/mobile_cap.stl"/>
+        <mesh filename="package://ros_pendulum/urdf/assets/mobile_cap.stl"/>
       </geometry>
       <material name="mobile_cap_material">
@@ -207,5 +207,5 @@
       <origin xyz="0 0 0" rpy="3.14159 0 0"/>
       <geometry>
-        <mesh filename="package://assets/mobile_cap.stl"/>
+        <mesh filename="package://ros_pendulum/urdf/assets/mobile_cap.stl"/>
       </geometry>
     </collision>
@@ -214,5 +214,5 @@
       <origin xyz="0 0 0" rpy="3.14159 0 0"/>
       <geometry>
-        <mesh filename="package://assets/mobile_handle.stl"/>
+        <mesh filename="package://ros_pendulum/urdf/assets/mobile_handle.stl"/>
       </geometry>
       <material name="mobile_handle_material">
@@ -223,5 +223,5 @@
       <origin xyz="0 0 0" rpy="3.14159 0 0"/>
       <geometry>
-        <mesh filename="package://assets/mobile_handle.stl"/>
+        <mesh filename="package://ros_pendulum/urdf/assets/mobile_handle.stl"/>
       </geometry>
     </collision>
@@ -230,5 +230,5 @@
       <origin xyz="0 0 0" rpy="3.14159 0 0"/>
       <geometry>
-        <mesh filename="package://assets/bearing_axe.stl"/>
+        <mesh filename="package://ros_pendulum/urdf/assets/bearing_axe.stl"/>
       </geometry>
       <material name="bearing_axe_material">
@@ -239,5 +239,5 @@
       <origin xyz="0 0 0" rpy="3.14159 0 0"/>
       <geometry>
-        <mesh filename="package://assets/bearing_axe.stl"/>
+        <mesh filename="package://ros_pendulum/urdf/assets/bearing_axe.stl"/>
       </geometry>
     </collision>
@@ -246,5 +246,5 @@
       <origin xyz="0.234 0 -0.0325" rpy="0 -1.5708 0"/>
       <geometry>
-        <mesh filename="package://assets/makerbeam_10mm.stl"/>
+        <mesh filename="package://ros_pendulum/urdf/assets/makerbeam_10mm.stl"/>
       </geometry>
       <material name="makerbeam_10mm_2_material">
@@ -255,5 +255,5 @@
       <origin xyz="0.234 0 -0.0325" rpy="0 -1.5708 0"/>
       <geometry>
-        <mesh filename="package://assets/makerbeam_10mm.stl"/>
+        <mesh filename="package://ros_pendulum/urdf/assets/makerbeam_10mm.stl"/>
       </geometry>
     </collision>
@@ -262,5 +262,5 @@
       <origin xyz="0 0 0" rpy="3.14159 0 0"/>
       <geometry>
-        <mesh filename="package://assets/mobile_spacer.stl"/>
+        <mesh filename="package://ros_pendulum/urdf/assets/mobile_spacer.stl"/>
       </geometry>
       <material name="mobile_spacer_material">
@@ -271,5 +271,5 @@
       <origin xyz="0 0 0" rpy="3.14159 0 0"/>
       <geometry>
-        <mesh filename="package://assets/mobile_spacer.stl"/>
+        <mesh filename="package://ros_pendulum/urdf/assets/mobile_spacer.stl"/>
       </geometry>
     </collision>
@@ -278,5 +278,5 @@
       <origin xyz="0 0 0" rpy="3.14159 0 0"/>
       <geometry>
-        <mesh filename="package://assets/magnet_stand.stl"/>
+        <mesh filename="package://ros_pendulum/urdf/assets/magnet_stand.stl"/>
       </geometry>
       <material name="magnet_stand_material">
@@ -287,5 +287,5 @@
       <origin xyz="0 0 0" rpy="3.14159 0 0"/>
       <geometry>
-        <mesh filename="package://assets/magnet_stand.stl"/>
+        <mesh filename="package://ros_pendulum/urdf/assets/magnet_stand.stl"/>
       </geometry>
     </collision>
@@ -294,5 +294,5 @@
       <origin xyz="0.246 0 0.011" rpy="-0 -0 -1.5708"/>
       <geometry>
-        <mesh filename="package://assets/wheel_support.stl"/>
+        <mesh filename="package://ros_pendulum/urdf/assets/wheel_support.stl"/>
       </geometry>
       <material name="wheel_support_material">
@@ -303,5 +303,5 @@
       <origin xyz="0.246 0 0.011" rpy="-0 -0 -1.5708"/>
       <geometry>
-        <mesh filename="package://assets/wheel_support.stl"/>
+        <mesh filename="package://ros_pendulum/urdf/assets/wheel_support.stl"/>
       </geometry>
     </collision>
@@ -318,5 +318,5 @@
       <origin xyz="0 0 0.0097" rpy="3.14159 0 -0"/>
       <geometry>
-        <mesh filename="package://assets/wheel.stl"/>
+        <mesh filename="package://ros_pendulum/urdf/assets/wheel.stl"/>
       </geometry>
       <material name="wheel_material">
@@ -327,5 +327,5 @@
       <origin xyz="0 0 0.0097" rpy="3.14159 0 -0"/>
       <geometry>
-        <mesh filename="package://assets/wheel.stl"/>
+        <mesh filename="package://ros_pendulum/urdf/assets/wheel.stl"/>
       </geometry>
     </collision>
