Commit message: Transmission, pos control

File: ros_pendulum/urdf/odrive_control.xacro (robot description, xacro)
@@ -12,6 +12,14 @@
         <state_interface name="position"/>
         <state_interface name="velocity"/>
-        <state_interface name="effort"/>s
+        <state_interface name="effort"/>
       </joint>
+      <transmission name="gim6010_transmission">
+        <plugin>transmission_interface/SimpleTransmission</plugin>
+        <actuator name="gim6010_motor" role="actuator1"/>
+        <joint name="gim6010" role="joint1">
+          <mechanical_reduction>8.0</mechanical_reduction>
+          <offset>0.0</offset>
+        </joint>
+      </transmission>
     </ros2_control>
   </xacro:macro>

File: ros_pendulum/urdf/robot.xacro (robot description, xacro)
@@ -300,5 +300,5 @@
     <limit lower="-100000.0" upper="100000.0" effort="400.0" velocity="100.0"/>
   </joint>
-  <xacro:include filename="$(find ros_pendulum)/urdf/odrive_control.xacro" />
+  <xacro:include filename="odrive_control.xacro" />
   <xacro:odrive_control />
 </robot>
