Commit message: Joint states aligned between real pendulum and isaaclab, training improved a bit

File: Pendulum/robot/robot.urdf (robot description, URDF)
Before this commit: robot robot, 3 links, 2 joints
Joints:
- joint gim6010: origin xyz=0.039 -0 -0 rpy=-0 1.5708 0 -> xyz=0.039 -0 -0 rpy=3.14159 1.5708 0

File: ros_pendulum/urdf/odrive_control.xacro (robot description, xacro)
@@ -20,5 +20,5 @@
         <joint name="gim6010" role="joint1">
           <mechanical_reduction>8.0</mechanical_reduction>
-          <offset>0.0</offset>
+          <offset>-0.24</offset>
         </joint>
       </transmission>

File: ros_pendulum/urdf/robot.xacro (robot description, xacro)
@@ -293,6 +293,6 @@
   <!-- Joint from housing to shaft -->
   <joint name="gim6010" type="revolute">
-    <!-- I had to change the pitch angle (-180 degrees) -->
-    <origin xyz="0.039 -0 -0" rpy="-0 -1.5708 0"/>
+    <!-- I had to change the roll angle (+180 degrees) otherwise mesh is swapped-->
+    <origin xyz="0.039 -0 -0" rpy="3.14159 1.5708 0"/>
     <parent link="housing"/>
     <child link="shaft"/>

Commit message: Add weight at the tip of the pole + RL experiments

File: Pendulum/robot/robot.urdf (robot description, URDF)
Before this commit: robot robot, 3 links, 2 joints
Links:
- added link motor_handle, mass 0.0902183; collision mesh filename=package://assets/as5600_breakout_board.stl; collision mesh filename=package://assets/bearing.stl
- added link wheel, mass 0.121; collision mesh filename=package://assets/wheel.stl; visual mesh filename=package://assets/wheel.stl
- link bearing_axe: mass 0.0589167 -> 0.063435; geometry collision mesh filename=package://assets/bearing_axe.stl; collision mesh filename=package://assets/magnet_stand.stl
- link shaft: mass 0.285218 -> 0.195; geometry collision mesh filename=package://assets/shaft.stl; visual mesh filename=package://assets/shaft.stl
Joints:
- added joint pole_to_wheel: type fixed, parent bearing_axe, child wheel, origin xyz=0.246 0 0.0207 rpy=3.14159 0 0, axis 0 0 1
- added joint shaft_to_mobile_handle: type fixed, parent shaft, child motor_handle, origin xyz=-0 0 -0.0015 rpy=0 -0 1.5708, axis 0 0 1
- joint free_0: limit lower=-100000.0 upper=100000.0 effort=400.0 velocity=100.0 -> lower=-100000.0 upper=100000.0 effort=100000.0 velocity=100000.0; origin xyz=0.241369 0 -0.0111 rpy=3.14159 -0 0 -> xyz=0 0.241369 -0.0096 rpy=-3.14159 0 1.5708; parent shaft -> motor_handle
- joint gim6010: limit lower=-100000.0 upper=100000.0 effort=400.0 velocity=100.0 -> lower=-100000.0 upper=100000.0 effort=100000.0 velocity=100000.0; origin xyz=0.039 -0 -0 rpy=3.14159 1.5708 0 -> xyz=0.039 -0 -0 rpy=-0 -1.5708 0

File: ros_pendulum/urdf/robot.xacro (robot description, xacro)
@@ -14,5 +14,5 @@
       <origin xyz="0 0 0" rpy="1.5708 0 -0"/>
       <geometry>
-        <mesh filename="package://ros_pendulum/urdf/assets/housing.stl"/>
+        <mesh filename="package://assets/housing.stl"/>
       </geometry>
       <material name="housing_material">
@@ -23,5 +23,5 @@
       <origin xyz="0 0 0" rpy="1.5708 0 -0"/>
       <geometry>
-        <mesh filename="package://ros_pendulum/urdf/assets/housing.stl"/>
+        <mesh filename="package://assets/housing.stl"/>
       </geometry>
     </collision>
@@ -30,13 +30,37 @@
   <link name="shaft">
     <inertial>
-      <origin xyz="0.0486873 -0 0.00116487" rpy="0 0 0"/>
-      <mass value="0.285218"/>
-      <inertia ixx="3.09982e-05" ixy="-0" ixz="8.46658e-05" iyy="0.0022823" iyz="0" izz="0.00229115"/>
+      <origin xyz="0 0 0.00431706" rpy="0 0 0"/>
+      <mass value="0.195"/>
+      <inertia ixx="1.74278e-05" ixy="0" ixz="-0" iyy="1.74278e-05" iyz="0" izz="3.04938e-05"/>
+    </inertial>
+    <!-- Part shaft -->
+    <visual>
+      <origin xyz="-0 0 0.039" rpy="0 1.5708 0"/>
+      <geometry>
+        <mesh filename="package://assets/shaft.stl"/>
+      </geometry>
+      <material name="shaft_material">
+        <color rgba="0.996078 0.996078 1 1"/>
+      </material>
+    </visual>
+    <collision>
+      <origin xyz="-0 0 0.039" rpy="0 1.5708 0"/>
+      <geometry>
+        <mesh filename="package://assets/shaft.stl"/>
+      </geometry>
+    </collision>
+  </link>
+  <!-- Link motor_handle -->
+  <link name="motor_handle">
+    <inertial>
+      <origin xyz="0 0.153921 -0.00414835" rpy="0 0 0"/>
+      <mass value="0.0902183"/>
+      <inertia ixx="0.000797422" ixy="-0" ixz="-0" iyy="7.44487e-06" iyz="-9.946e-06" izz="0.000799332"/>
     </inertial>
     <!-- Part motor_handle -->
     <visual>
-      <origin xyz="-0 0 0.0392" rpy="-0 1.5708 0"/>
-      <geometry>
-        <mesh filename="package://ros_pendulum/urdf/assets/motor_handle.stl"/>
+      <origin xyz="-0 -0 0.0437" rpy="-1.5708 1.5708 0"/>
+      <geometry>
+        <mesh filename="package://assets/motor_handle.stl"/>
       </geometry>
       <material name="motor_handle_material">
@@ -45,14 +69,14 @@
     </visual>
     <collision>
-      <origin xyz="-0 0 0.0392" rpy="-0 1.5708 0"/>
-      <geometry>
-        <mesh filename="package://ros_pendulum/urdf/assets/motor_handle.stl"/>
+      <origin xyz="-0 -0 0.0437" rpy="-1.5708 1.5708 0"/>
+      <geometry>
+        <mesh filename="package://assets/motor_handle.stl"/>
       </geometry>
     </collision>
     <!-- Part bearing -->
     <visual>
-      <origin xyz="0.241369 0 -0.0111" rpy="-0 0 0"/>
-      <geometry>
-        <mesh filename="package://ros_pendulum/urdf/assets/bearing.stl"/>
+      <origin xyz="0 0.241369 -0.0096" rpy="0 0 1.5708"/>
+      <geometry>
+        <mesh filename="package://assets/bearing.stl"/>
       </geometry>
       <material name="bearing_material">
@@ -61,14 +85,14 @@
     </visual>
     <collision>
-      <origin xyz="0.241369 0 -0.0111" rpy="-0 0 0"/>
-      <geometry>
-        <mesh filename="package://ros_pendulum/urdf/assets/bearing.stl"/>
+      <origin xyz="0 0.241369 -0.0096" rpy="0 0 1.5708"/>
+      <geometry>
+        <mesh filename="package://assets/bearing.stl"/>
       </geometry>
     </collision>
     <!-- Part encoder_plate -->
     <visual>
-      <origin xyz="0.241369 0 -0.0111" rpy="-0 0 0"/>
-      <geometry>
-        <mesh filename="package://ros_pendulum/urdf/assets/encoder_plate.stl"/>
+      <origin xyz="0 0.241369 -0.0096" rpy="0 0 1.5708"/>
+      <geometry>
+        <mesh filename="package://assets/encoder_plate.stl"/>
       </geometry>
       <material name="encoder_plate_material">
@@ -77,14 +101,14 @@
     </visual>
     <collision>
-      <origin xyz="0.241369 0 -0.0111" rpy="-0 0 0"/>
-      <geometry>
-        <mesh filename="package://ros_pendulum/urdf/assets/encoder_plate.stl"/>
+      <origin xyz="0 0.241369 -0.0096" rpy="0 0 1.5708"/>
+      <geometry>
+        <mesh filename="package://assets/encoder_plate.stl"/>
       </geometry>
     </collision>
     <!-- Part fixed_handle -->
     <visual>
-      <origin xyz="0.241369 0 -0.0111" rpy="-0 0 0"/>
-      <geometry>
-        <mesh filename="package://ros_pendulum/urdf/assets/fixed_handle.stl"/>
+      <origin xyz="0 0.241369 -0.0096" rpy="0 0 1.5708"/>
+      <geometry>
+        <mesh filename="package://assets/fixed_handle.stl"/>
       </geometry>
       <material name="fixed_handle_material">
@@ -93,30 +117,14 @@
     </visual>
     <collision>
-      <origin xyz="0.241369 0 -0.0111" rpy="-0 0 0"/>
-      <geometry>
-        <mesh filename="package://ros_pendulum/urdf/assets/fixed_handle.stl"/>
-      </geometry>
-    </collision>
-    <!-- Part shaft -->
-    <visual>
-      <origin xyz="0 -0 0.039" rpy="3.14159 1.5708 0"/>
-      <geometry>
-        <mesh filename="package://ros_pendulum/urdf/assets/shaft.stl"/>
-      </geometry>
-      <material name="shaft_material">
-        <color rgba="0.996078 0.996078 1 1"/>
-      </material>
-    </visual>
-    <collision>
-      <origin xyz="0 -0 0.039" rpy="3.14159 1.5708 0"/>
-      <geometry>
-        <mesh filename="package://ros_pendulum/urdf/assets/shaft.stl"/>
+      <origin xyz="0 0.241369 -0.0096" rpy="0 0 1.5708"/>
+      <geometry>
+        <mesh filename="package://assets/fixed_handle.stl"/>
       </geometry>
     </collision>
     <!-- Part fixed_cap -->
     <visual>
-      <origin xyz="0.241369 0 -0.0111" rpy="-0 0 0"/>
-      <geometry>
-        <mesh filename="package://ros_pendulum/urdf/assets/fixed_cap.stl"/>
+      <origin xyz="0 0.241369 -0.0096" rpy="0 0 1.5708"/>
+      <geometry>
+        <mesh filename="package://assets/fixed_cap.stl"/>
       </geometry>
       <material name="fixed_cap_material">
@@ -125,14 +133,14 @@
     </visual>
     <collision>
-      <origin xyz="0.241369 0 -0.0111" rpy="-0 0 0"/>
-      <geometry>
-        <mesh filename="package://ros_pendulum/urdf/assets/fixed_cap.stl"/>
+      <origin xyz="0 0.241369 -0.0096" rpy="0 0 1.5708"/>
+      <geometry>
+        <mesh filename="package://assets/fixed_cap.stl"/>
       </geometry>
     </collision>
     <!-- Part encoder_plate_spacer -->
     <visual>
-      <origin xyz="0.241369 0 -0.0111" rpy="-0 0 0"/>
-      <geometry>
-        <mesh filename="package://ros_pendulum/urdf/assets/encoder_plate_spacer.stl"/>
+      <origin xyz="0 0.241369 -0.0096" rpy="0 0 1.5708"/>
+      <geometry>
+        <mesh filename="package://assets/encoder_plate_spacer.stl"/>
       </geometry>
       <material name="encoder_plate_spacer_material">
@@ -141,14 +149,14 @@
     </visual>
     <collision>
-      <origin xyz="0.241369 0 -0.0111" rpy="-0 0 0"/>
-      <geometry>
-        <mesh filename="package://ros_pendulum/urdf/assets/encoder_plate_spacer.stl"/>
+      <origin xyz="0 0.241369 -0.0096" rpy="0 0 1.5708"/>
+      <geometry>
+        <mesh filename="package://assets/encoder_plate_spacer.stl"/>
       </geometry>
     </collision>
     <!-- Part as5600_breakout_board -->
     <visual>
-      <origin xyz="0.241369 0 -0.0111" rpy="-0 0 0"/>
-      <geometry>
-        <mesh filename="package://ros_pendulum/urdf/assets/as5600_breakout_board.stl"/>
+      <origin xyz="0 0.241369 -0.0096" rpy="0 0 1.5708"/>
+      <geometry>
+        <mesh filename="package://assets/as5600_breakout_board.stl"/>
       </geometry>
       <material name="as5600_breakout_board_material">
@@ -157,14 +165,14 @@
     </visual>
     <collision>
-      <origin xyz="0.241369 0 -0.0111" rpy="-0 0 0"/>
-      <geometry>
-        <mesh filename="package://ros_pendulum/urdf/assets/as5600_breakout_board.stl"/>
+      <origin xyz="0 0.241369 -0.0096" rpy="0 0 1.5708"/>
+      <geometry>
+        <mesh filename="package://assets/as5600_breakout_board.stl"/>
       </geometry>
     </collision>
     <!-- Part makerbeam_10mm -->
     <visual>
-      <origin xyz="-0 0 0.0392" rpy="-0 1.5708 0"/>
-      <geometry>
-        <mesh filename="package://ros_pendulum/urdf/assets/makerbeam_10mm.stl"/>
+      <origin xyz="0 -0 0.0437" rpy="-1.5708 1.5708 0"/>
+      <geometry>
+        <mesh filename="package://assets/makerbeam_10mm.stl"/>
       </geometry>
       <material name="makerbeam_10mm_material">
@@ -173,7 +181,7 @@
     </visual>
     <collision>
-      <origin xyz="-0 0 0.0392" rpy="-0 1.5708 0"/>
-      <geometry>
-        <mesh filename="package://ros_pendulum/urdf/assets/makerbeam_10mm.stl"/>
+      <origin xyz="0 -0 0.0437" rpy="-1.5708 1.5708 0"/>
+      <geometry>
+        <mesh filename="package://assets/makerbeam_10mm.stl"/>
       </geometry>
     </collision>
@@ -182,13 +190,13 @@
   <link name="bearing_axe">
     <inertial>
-      <origin xyz="0.0670267 9.60394e-06 0.0137414" rpy="0 0 0"/>
-      <mass value="0.0589167"/>
-      <inertia ixx="6.41916e-06" ixy="3.0456e-08" ixz="-9.18141e-06" iyy="0.000344996" iyz="-1.195e-09" izz="0.00034346"/>
+      <origin xyz="0.0790606 8.91988e-06 0.0137513" rpy="0 0 0"/>
+      <mass value="0.063435"/>
+      <inertia ixx="6.66733e-06" ixy="3.7265e-08" ixz="-9.81805e-06" iyy="0.00046914" iyz="-1.189e-09" izz="0.000467602"/>
     </inertial>
     <!-- Part mobile_cap -->
     <visual>
-      <origin xyz="0 0 0" rpy="-3.14159 -0 -0"/>
-      <geometry>
-        <mesh filename="package://ros_pendulum/urdf/assets/mobile_cap.stl"/>
+      <origin xyz="0 0 0" rpy="3.14159 0 0"/>
+      <geometry>
+        <mesh filename="package://assets/mobile_cap.stl"/>
       </geometry>
       <material name="mobile_cap_material">
@@ -197,14 +205,14 @@
     </visual>
     <collision>
-      <origin xyz="0 0 0" rpy="-3.14159 -0 -0"/>
-      <geometry>
-        <mesh filename="package://ros_pendulum/urdf/assets/mobile_cap.stl"/>
+      <origin xyz="0 0 0" rpy="3.14159 0 0"/>
+      <geometry>
+        <mesh filename="package://assets/mobile_cap.stl"/>
       </geometry>
     </collision>
     <!-- Part mobile_handle -->
     <visual>
-      <origin xyz="0 0 0" rpy="-3.14159 -0 -0"/>
-      <geometry>
-        <mesh filename="package://ros_pendulum/urdf/assets/mobile_handle.stl"/>
+      <origin xyz="0 0 0" rpy="3.14159 0 0"/>
+      <geometry>
+        <mesh filename="package://assets/mobile_handle.stl"/>
       </geometry>
       <material name="mobile_handle_material">
@@ -213,14 +221,14 @@
     </visual>
     <collision>
-      <origin xyz="0 0 0" rpy="-3.14159 -0 -0"/>
-      <geometry>
-        <mesh filename="package://ros_pendulum/urdf/assets/mobile_handle.stl"/>
+      <origin xyz="0 0 0" rpy="3.14159 0 0"/>
+      <geometry>
+        <mesh filename="package://assets/mobile_handle.stl"/>
       </geometry>
     </collision>
     <!-- Part bearing_axe -->
     <visual>
-      <origin xyz="0 0 0" rpy="-3.14159 -0 -0"/>
-      <geometry>
-        <mesh filename="package://ros_pendulum/urdf/assets/bearing_axe.stl"/>
+      <origin xyz="0 0 0" rpy="3.14159 0 0"/>
+      <geometry>
+        <mesh filename="package://assets/bearing_axe.stl"/>
       </geometry>
       <material name="bearing_axe_material">
@@ -229,14 +237,14 @@
     </visual>
     <collision>
-      <origin xyz="0 0 0" rpy="-3.14159 -0 -0"/>
-      <geometry>
-        <mesh filename="package://ros_pendulum/urdf/assets/bearing_axe.stl"/>
+      <origin xyz="0 0 0" rpy="3.14159 0 0"/>
+      <geometry>
+        <mesh filename="package://assets/bearing_axe.stl"/>
       </geometry>
     </collision>
     <!-- Part makerbeam_10mm_2 -->
     <visual>
-      <origin xyz="0.234 -0 -0.0295" rpy="0 -1.5708 0"/>
-      <geometry>
-        <mesh filename="package://ros_pendulum/urdf/assets/makerbeam_10mm.stl"/>
+      <origin xyz="0.234 0 -0.0325" rpy="0 -1.5708 0"/>
+      <geometry>
+        <mesh filename="package://assets/makerbeam_10mm.stl"/>
       </geometry>
       <material name="makerbeam_10mm_2_material">
@@ -245,14 +253,14 @@
     </visual>
     <collision>
-      <origin xyz="0.234 -0 -0.0295" rpy="0 -1.5708 0"/>
-      <geometry>
-        <mesh filename="package://ros_pendulum/urdf/assets/makerbeam_10mm.stl"/>
+      <origin xyz="0.234 0 -0.0325" rpy="0 -1.5708 0"/>
+      <geometry>
+        <mesh filename="package://assets/makerbeam_10mm.stl"/>
       </geometry>
     </collision>
     <!-- Part mobile_spacer -->
     <visual>
-      <origin xyz="0 0 0" rpy="-3.14159 -0 -0"/>
-      <geometry>
-        <mesh filename="package://ros_pendulum/urdf/assets/mobile_spacer.stl"/>
+      <origin xyz="0 0 0" rpy="3.14159 0 0"/>
+      <geometry>
+        <mesh filename="package://assets/mobile_spacer.stl"/>
       </geometry>
       <material name="mobile_spacer_material">
@@ -261,14 +269,14 @@
     </visual>
     <collision>
-      <origin xyz="0 0 0" rpy="-3.14159 -0 -0"/>
-      <geometry>
-        <mesh filename="package://ros_pendulum/urdf/assets/mobile_spacer.stl"/>
+      <origin xyz="0 0 0" rpy="3.14159 0 0"/>
+      <geometry>
+        <mesh filename="package://assets/mobile_spacer.stl"/>
       </geometry>
     </collision>
     <!-- Part magnet_stand -->
     <visual>
-      <origin xyz="0 0 0" rpy="-3.14159 -0 -0"/>
-      <geometry>
-        <mesh filename="package://ros_pendulum/urdf/assets/magnet_stand.stl"/>
+      <origin xyz="0 0 0" rpy="3.14159 0 0"/>
+      <geometry>
+        <mesh filename="package://assets/magnet_stand.stl"/>
       </geometry>
       <material name="magnet_stand_material">
@@ -277,26 +285,79 @@
     </visual>
     <collision>
-      <origin xyz="0 0 0" rpy="-3.14159 -0 -0"/>
-      <geometry>
-        <mesh filename="package://ros_pendulum/urdf/assets/magnet_stand.stl"/>
-      </geometry>
-    </collision>
-  </link>
-  <!-- Joint from shaft to bearing_axe -->
+      <origin xyz="0 0 0" rpy="3.14159 0 0"/>
+      <geometry>
+        <mesh filename="package://assets/magnet_stand.stl"/>
+      </geometry>
+    </collision>
+    <!-- Part wheel_support -->
+    <visual>
+      <origin xyz="0.246 0 0.011" rpy="-0 -0 -1.5708"/>
+      <geometry>
+        <mesh filename="package://assets/wheel_support.stl"/>
+      </geometry>
+      <material name="wheel_support_material">
+        <color rgba="0.615686 0.811765 0.929412 1"/>
+      </material>
+    </visual>
+    <collision>
+      <origin xyz="0.246 0 0.011" rpy="-0 -0 -1.5708"/>
+      <geometry>
+        <mesh filename="package://assets/wheel_support.stl"/>
+      </geometry>
+    </collision>
+  </link>
+  <!-- Link wheel -->
+  <link name="wheel">
+    <inertial>
+      <origin xyz="0 -0 -0.0182091" rpy="0 0 0"/>
+      <mass value="0.121"/>
+      <inertia ixx="5.25074e-05" ixy="0" ixz="0" iyy="5.25074e-05" iyz="-0" izz="7.43868e-05"/>
+    </inertial>
+    <!-- Part wheel -->
+    <visual>
+      <origin xyz="0 0 0.0097" rpy="3.14159 0 -0"/>
+      <geometry>
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